File: PhonieBoxHat.sch (KiCad schematic (older format))
At the start: 33 parts, among them J1 Raspberry_Pi_2_3, J2 Display, J3 OnOffShim, J4 VOL-, J5 VOL+, J6 Prev, J7 Play/Pause, J8 Next, J9 PowerLed

Commit message: v0.3
New version of the PCB to integrate the OnOffShim
Parts:
- removed J2: Display, Connector_PinHeader_2.54mm:PinHeader_2x02_P2.54mm_Horizontal, symbol Connector:Conn_01x04_Male
- removed J3: OnOffShim, Connector_PinHeader_2.54mm:PinHeader_2x02_P2.54mm_Horizontal, symbol Connector:Conn_01x04_Male
- removed J4: VOL-, Connector_PinHeader_2.54mm:PinHeader_2x02_P2.54mm_Horizontal, symbol Connector:Conn_01x04_Male
- removed J5: VOL+, Connector_PinHeader_2.54mm:PinHeader_2x02_P2.54mm_Horizontal, symbol Connector:Conn_01x04_Male
- removed J6: Prev, Connector_PinHeader_2.54mm:PinHeader_2x02_P2.54mm_Horizontal, symbol Connector:Conn_01x04_Male
- removed J7: Play/Pause, Connector_PinHeader_2.54mm:PinHeader_2x02_P2.54mm_Horizontal, symbol Connector:Conn_01x04_Male
- removed J8: Next, Connector_PinHeader_2.54mm:PinHeader_2x02_P2.54mm_Horizontal, symbol Connector:Conn_01x04_Male
- added J10: Buttons, Connector_PinHeader_2.54mm:PinHeader_2x12_P2.54mm_Horizontal, symbol Connector_Generic:Conn_02x12_Odd_Even
- added J2: OnOffShim, Connector_PinHeader_2.54mm:PinHeader_2x06_P2.54mm_Vertical, symbol Connector_Generic:Conn_02x06_Odd_Even
- added J3: PWR BTN, Connector_PinSocket_2.54mm:PinSocket_1x02_P2.54mm_Vertical, symbol Connector:Conn_01x02_Male
Connections:
- wire segments 77 -> 68
- no-connect marks 28 -> 38
Other:
- moved on the sheet: J9, R1, R10, R11, R12, R13, R14, R15, R16, R2, R3, R4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
